File: sig_scan_pcb/sig_scan_pcb.kicad_sch (KiCad schematic)
At the start: 0 parts

Commit message: adding uncompleet rtl-sdr design
Parts:
- added AE1: Antenna_Shield, RF_Antenna:Texas_SWRA117D_2.4GHz_Left, symbol Device:Antenna_Shield
- added C1, C2: 10uF, Capacitor_SMD:C_0805_2012Metric_Pad1.18x1.45mm_HandSolder, symbol Device:C_Small
- added C10, C13, C22, C25, C27: 27pF, symbol Device:C_Small
- added C11, C23, C24: 10pF, Capacitor_SMD:C_0805_2012Metric_Pad1.18x1.45mm_HandSolder, symbol Device:C_Small
- added C12: 1uF, Capacitor_SMD:C_0805_2012Metric_Pad1.18x1.45mm_HandSolder, symbol Device:C_Small
- added C14, C9: 104, symbol Device:C_Small
- added C15: 22uF 16v Cer, symbol Device:C_Polarized_Small
- added C16: 10uF 16v Cer, symbol Device:C_Polarized_Small
- added C17, C20, C21: 100nF 16v Cer, symbol Device:C_Polarized_Small
- added C18, C19: 47pF, symbol Device:C_Small
- added C26: 100nF, symbol Device:C_Polarized_Small
- added C3: C_Small, symbol Device:C_Small
- added C31, C34, C38: 1uF, Capacitor_SMD:C_0805_2012Metric, symbol Device:C_Small
- added C32: 10nF, Capacitor_SMD:C_0805_2012Metric, symbol Device:C_Small
- added C33: 10uF, Capacitor_SMD:C_0805_2012Metric, symbol Device:C_Small
- added C35, C36, C37, C39, C40: 100nF, Capacitor_SMD:C_0805_2012Metric, symbol Device:C_Small
- added C4, C7: DNP, Capacitor_SMD:C_0805_2012Metric_Pad1.18x1.45mm_HandSolder, symbol Device:C_Small
- added C42, C43, C45: C_Small, Capacitor_SMD:C_0805_2012Metric, symbol Device:C_Small
- added C5, C6: 22uF, Capacitor_SMD:C_0805_2012Metric_Pad1.18x1.45mm_HandSolder, symbol Device:C_Small
- added C8: 105, symbol Device:C_Small
- added D1, D2: 1N4148W, Diode_SMD:D_SOD-123, symbol Diode:1N4148W
- added D3, D4: Diod, symbol Device:D_Small
- added IC1: AZ1117H-3.3TRE1, AZ1117H-3_3TRE1:SOT230P700X180-4N, symbol AZ1117H-3_3TRE1:AZ1117H-3.3TRE1
- added J1: 12V Connector, TerminalBlock:TerminalBlock_bornier-2_P5.08mm, symbol Connector:Conn_01x02_Pin
- added J10, J4: LED Connector, Connector_PinHeader_2.54mm:PinHeader_1x02_P2.54mm_Vertical, symbol Connector:Conn_01x02_Pin
- added J12: PROG, Connector_PinHeader_2.54mm:PinHeader_1x04_P2.54mm_Vertical, symbol Connector:Conn_01x04_Pin
- added J13: GPIO Connector, Connector_PinHeader_2.54mm:PinHeader_2x15_P2.54mm_Vertical, symbol Connector_Generic:Conn_02x15_Odd_Even
- added J15: I/O Connector, Connector_PinHeader_2.54mm:PinHeader_2x08_P2.54mm_Vertical, symbol Connector_Generic:Conn_02x08_Odd_Even
- added J16: Screw_Terminal_01x03, TerminalBlock:TerminalBlock_bornier-3_P5.08mm, symbol Connector:Screw_Terminal_01x03
- added J17: Screw_Terminal_01x04, TerminalBlock:TerminalBlock_bornier-4_P5.08mm, symbol Connector:Screw_Terminal_01x04
- added J2: UJ20-C-H-G-SMT-P16-TR, Connector_USB:USB_C_Receptacle_G-Switch_GT-USB-7010ASV, symbol Connector:USB_C_Receptacle_USB2.0_16P
- added J3: USB Switch, Connector_PinHeader_2.54mm:PinHeader_1x03_P2.54mm_Vertical, symbol Connector:Conn_01x03_Pin
- added J5: Conn_Coaxial, symbol Connector:Conn_Coaxial
- added JP6, JP8: SP, Jumper:SolderJumper-3_P1.3mm_Bridged12_RoundedPad1.0x1.5mm, symbol Jumper:SolderJumper_3_Bridged12
- added L1: 24nH, Inductor_SMD:L_0805_2012Metric_Pad1.15x1.40mm_HandSolder, symbol Device:L_Small
- added L2: 2nH, Inductor_SMD:L_0603_1608Metric, symbol Device:L_Small
- added L3, L4: L_Small, Inductor_SMD:L_0805_2012Metric, symbol Device:L_Small
- added L5: L_Small, symbol Device:L_Small
- added L6, L7: 150nH, symbol Device:L
- added L8: 4.7uH, symbol Device:L
- added L9: beet, symbol Device:L_Ferrite_Small
- added R1, R6: 10k, symbol Device:R_Small
- added R10: 103, symbol Device:R_Small
- added R11, R12, R26: 10K, Resistor_SMD:R_0805_2012Metric_Pad1.20x1.40mm_HandSolder, symbol Device:R_Small
- added R13: 101, symbol Device:R_Small
- added R14, R16, R8, R9: 220, symbol Device:R_Small
- added R15, R17: 472, symbol Device:R_Small
- added R2, R5: 5K1, Resistor_SMD:R_0805_2012Metric_Pad1.20x1.40mm_HandSolder, symbol Device:R_Small
- added R22, R23, R36, R37: 4K7, Resistor_SMD:R_0805_2012Metric_Pad1.20x1.40mm_HandSolder, symbol Device:R_Small
- added R27: 6K8, Resistor_SMD:R_0805_2012Metric_Pad1.20x1.40mm_HandSolder, symbol Device:R_Small
- added R3, R4: 0, Resistor_SMD:R_0805_2012Metric_Pad1.20x1.40mm_HandSolder, symbol Device:R_Small
- added R33: 499, Resistor_SMD:R_0805_2012Metric_Pad1.20x1.40mm_HandSolder, symbol Device:R_Small
- added R34, R7: 220, Resistor_SMD:R_0805_2012Metric_Pad1.20x1.40mm_HandSolder, symbol Device:R_Small
- added SW1: BOOT, Button_Switch_SMD:SW_Tactile_SPST_NO_Straight_CK_PTS636Sx25SMTRLFS, symbol Switch:SW_Push
- added SW2: RESET, Button_Switch_SMD:SW_Tactile_SPST_NO_Straight_CK_PTS636Sx25SMTRLFS, symbol Switch:SW_Push
- added U1: AZ1117H-5.0TRE1, AZ1117H-5.0TRE1:SOT230P700X180-4N, symbol AZ1117H-5.0TRE1:AZ1117H-5.0TRE1
- added U2: RTL2832U, RTL2832U:QFN40P600X600X100-49N, symbol RTL2832U:RTL2832U
- added U3: R820T, R820T:QFN50P400X400X90-25N, symbol R820T:R820T
- added U4: ESP32-S3FN8, Package_DFN_QFN:QFN-56-1EP_7x7mm_P0.4mm_EP4x4mm, symbol MCU_Espressif:ESP32-S3
- added U5: M24C02-WMN, Package_SO:SOIC-8_3.9x4.9mm_P1.27mm, symbol Memory_EEPROM:M24C02-WMN
- added Y1: 40MHz, ABM8-40.000MHZ-10-B1U-T:ABM810000MHZ12D2W, symbol Device:Crystal_GND24_Small
- added Y2: 16MHz, symbol Device:Crystal_Small
- added Y3: 28.8Mhz, symbol Device:Crystal_Small
Connections:
- new net: C16.1, C17.1, C20.1, L9.1, U2.25 (SW_VDD3), U2.26 (SW_VDD3)
- new net: JP8.2 (C), R37.1
- new net: R37.2, U4.52 (GPIO46)
- new net: C23.2, L1.1, Y1.1
- new net: J4.1 (Pin_1), R7.1
- new net: C45.1, L4.2
- new net: R16.2, R17.2, U2.17 (I2C_SDAT)
- new net: R16.1, U3.7 (SDA)
- new net: C8.1, U3.4 (DET1)
- new net: C15.1, L8.1, U2.23 (FB)
- new net: R26.1, R27.2, U4.24 (GPIO18)
- new net: C25.1, R8.2
- new net: C25.2, U2.1 (VIP)
- new net: AE1.1 (A), C43.1, L3.2, L4.1
- new net: R14.1, U3.6 (SCL)
- new net: R14.2, R15.2, U2.16 (I2C_SCLT)
- new net: C38.1, C39.1, U4.29 (VDD_SPI)
- new net: D1.2 (A), J1.1 (Pin_1)
- new net: C19.2, Y3.1
- new net: C18.2, Y3.2
- new net: C3.2, L5.1
- new net: L5.2, U3.24 (RF_IN)
- new net: C24.2, U4.53 (XTAL_N), Y1.3
- new net: R8.1, U3.13 (IF_P)
- new net: C36.2, L2.2, U4.2 (VDD3P3), U4.3 (VDD3P3)
- new net: R33.1, U4.49 (U0TXD)
- new net: J12.3 (Pin_3), R33.2
- new net: L6.1, U3.20 (TF2P)
- new net: L6.2, U3.22 (TF1P)
- new net: C14.1, R10.1, U3.14 (IF_AGC)
- new net: R10.2, U2.13 (AGC_IF)
- new net: J10.1 (Pin_1), R34.1
- new net: R13.2, U2.10 (XO)
- new net: C27.2, R13.1, U2.11 (XI)
- new net: C22.2, U2.2 (VIN)
- new net: L8.2, U2.24 (REG_OUT)
- new net: J2.A5 (CC1), R2.1
- new net: J2.A6 (D+), J2.B6 (D+), R4.1
- new net: J2.A7 (D-), J2.B7 (D-), R3.1
- new net: J2.B5 (CC2), R5.1
- new net: C27.1, U3.10 (CLK_OUT)
- new net: C10.1, U3.8 (XTAL_I), Y2.1
- new net: C13.1, U3.9 (XTAL_O), Y2.2
- new net: C3.1, D3.2 (A), D4.1 (K), J5.1 (In)
- new net: R9.1, U3.12 (IF_N)
- new net: C22.1, R9.2
- new net: JP6.2 (C), R36.1
- new net: R36.2, U4.51 (GPIO45)
- new net: J12.2 (Pin_2), U4.50 (U0RXD)
- new net: D2.2 (A), J3.3 (Pin_3)
- new net: L1.2, U4.54 (XTAL_P)
- new net: C42.1, L3.1, U4.1 (LNA_IN)
- new net: L7.1, U3.19 (TF2N)
- new net: L7.2, U3.21 (TF1N)
- new net: C9.1, U3.5 (DET2)
- new net +15V: C1.2, C2.2, D1.1 (K), D2.1 (K), IC1.3 (INPUT), U1.3 (INPUT)
- new net +3.3V: C21.1, C26.1, C31.2, C32.2, C33.2, C34.2, C35.2, C37.1, C40.1, C5.2, IC1.2 (OUTPUT), IC1.4 (VOUT), J12.4 (Pin_4), J13.1 (Pin_1), J4.2 (Pin_2), JP6.3 (B), JP8.3 (B), L2.1, L9.2, R1.1, R11.2, R12.2, R15.1, R17.1, R22.2, R23.2, R6.1, U3.11 (VCC), U3.2 (VCC), U3.23 (VCC), U4.20 (VDD3P3_RTC), U4.46 (VDD3P3_CPU), U4.55 (VDDA), U4.56 (VDDA), U5.8 (VCC)
- new net +5V: C6.2, J13.4 (Pin_4), J3.1 (Pin_1), U1.2 (OUTPUT), U1.4 (VOUT)
- new net CHIP_PU: C12.2, R12.1, SW2.2, U4.4 (CHIP_PU)
- new net EXP GND: J17.4 (Pin_4)
- new net GND: AE1.2 (Shield), C1.1, C10.2, C11.1, C12.1, C13.2, C14.2, C15.2, C16.2, C17.2, C18.1, C19.1, C2.1, C20.2, C21.2, C23.1, C24.1, C26.2, C31.1, C32.1, C33.1, C34.1, C35.1, C36.1, C37.2, C38.2, C39.2, C4.2, C40.2, C42.2, C43.2, C45.2, C5.1, C6.1, C7.2, C8.2, C9.2, D3.1 (K), D4.2 (A), IC1.1 (GND), J1.2 (Pin_2), J12.1 (Pin_1), J13.2 (Pin_2), J15.10 (Pin_10), J15.12 (Pin_12), J15.14 (Pin_14), J15.16 (Pin_16), J15.2 (Pin_2), J15.4 (Pin_4), J15.6 (Pin_6), J15.8 (Pin_8), J2.A1 (GND), J2.A12 (GND), J2.B1 (GND), J2.B12 (GND), J2.S1 (SHIELD), J5.2 (Ext), JP6.1 (A), JP8.1 (A), R2.2, R27.1, R34.2, R5.2, R7.2, SW1.1, SW2.1, U1.1 (ADJ/GND), U2.49 (GND), U3.16 (GND), U3.25 (GND), U4.57 (GND), U5.1 (E0), U5.2 (E1), U5.3 (E2), U5.4 (VSS), Y1.2, Y1.4
- new net GNDA: U2.3 (GNDA), U2.45 (GNDA)
- new net GPIO0: C11.2, R11.1, SW1.2, U4.5 (GPIO0)
- new net GPIO1: J13.11 (Pin_11), U4.6 (GPIO1)
- new net GPIO10: J13.21 (Pin_21), U4.15 (GPIO10)
- new net GPIO11: J13.15 (Pin_15), U4.16 (GPIO11)
- new net GPIO12: J13.13 (Pin_13), U4.17 (GPIO12)
- new net GPIO13: J13.18 (Pin_18), U4.18 (GPIO13)
- new net GPIO14: J13.17 (Pin_17), U4.19 (GPIO14)
- new net GPIO15: J13.22 (Pin_22), U4.21 (XTAL_32K_P)
- new net GPIO16: J13.19 (Pin_19), U4.22 (XTAL_32K_N)
- new net GPIO17: J13.20 (Pin_20), U4.23 (GPIO17)
- new net GPIO21: J13.23 (Pin_23), U4.27 (GPIO21)
- new net GPIO2/PTT ESP: J13.12 (Pin_12), U4.7 (GPIO2)
- new net GPIO3: J13.9 (Pin_9), U4.8 (GPIO3)
- new net GPIO38: J13.26 (Pin_26), U4.43 (GPIO38)
- new net GPIO39/MTCK: J13.28 (Pin_28), U4.44 (MTCK)
- new net GPIO40/MTDO: J13.30 (Pin_30), U4.45 (MTDO)
- new net GPIO41/MTDI: J13.29 (Pin_29), U4.47 (MTDI)
- new net GPIO42/MTMS: J13.27 (Pin_27), U4.48 (MTMS)
- new net GPIO47: J13.25 (Pin_25), U4.37 (SPICLK_P)
- new net GPIO48: J10.2 (Pin_2), J13.24 (Pin_24), U4.36 (SPICLK_N)
- new net GPIO4/BCLK: J13.10 (Pin_10), U4.9 (GPIO4)
- new net GPIO5/FSYNC: J13.7 (Pin_7), U4.10 (GPIO5)
- new net GPIO6/DOUT: J13.8 (Pin_8), U4.11 (GPIO6)
- new net GPIO7/DIN: J13.5 (Pin_5), U4.12 (GPIO7)
- new net IN1M: J15.5 (Pin_5)
- new net IN1P: J15.7 (Pin_7)
- new net IN2M: J15.1 (Pin_1)
- new net IN2P: J15.3 (Pin_3)
- new net Mic GND: J16.2 (Pin_2)
- new net OUT1M: J15.15 (Pin_15)
- new net OUT1P: J15.9 (Pin_9)
- new net OUT2M: J15.11 (Pin_11)
- new net OUT2P: J15.13 (Pin_13)
- new net PTT: J17.2 (Pin_2)
- new net PTT GND: J17.1 (Pin_1)
- new net PTT Power: J17.3 (Pin_3)
- new net Radio EXP: J16.1 (Pin_1)
- new net Radio Mic: J16.3 (Pin_3)
- new net SCL: J13.6 (Pin_6), R22.1, R6.2, U2.18 (I2C_SCL), U4.14 (GPIO9), U5.6 (SCL)
- new net SDA: J13.3 (Pin_3), R1.2, R23.1, U2.19 (I2C_SDA), U4.13 (GPIO8), U5.5 (SDA)
- new net USBD+: C4.1, J13.14 (Pin_14), R4.2, U4.26 (GPIO20/USB_D+)
- new net USBD-: C7.1, J13.16 (Pin_16), R3.2, U4.25 (GPIO19/USB_D-)
- new net VBUS: J2.A4 (VBUS), J2.A9 (VBUS), J2.B4 (VBUS), J2.B9 (VBUS), J3.2 (Pin_2), R26.2
- no-connect marks 0 -> 14
Other:
- note added: "Check connections"
- note added: "EXP GND"
- note added: "Mic GND"
- note added: "PTT"
- note added: "PTT Power"
- note added: "PTTGND"
- note added: "Radio EXP"
- note added: "Radio Mic"
- company: (none) -> Giga Technology
- title: (none) -> Sig Scan

Commit message: almost compleet design needs psu
Parts:
- added C28, C49, C50, C51, C52, C53, C55, C56, C57: 100nF, symbol Device:C_Small
- added C29, C30, C41: 105, symbol Device:C_Small
- added C44, C46: 27pF, symbol Device:C_Small
- added C47, C48: 1Uf, symbol Device:C_Small
- added C54: 1uF, symbol Device:C_Small
- added J6: CLK TP, symbol Connector:Conn_01x01_Pin
- added R18: 10k, symbol Device:R_Small
- added R19: 1K, symbol Device:R_Small
- added R20: 220, Resistor_SMD:R_0805_2012Metric_Pad1.20x1.40mm_HandSolder, symbol Device:R_Small
- added U6: RA-02_LORA, RA-02_LORA:MODULE_RA-02_LORA, symbol RA-02-lora:RA-02_LORA
- C3: value C_Small -> 1uF
- L5: value L_Small -> 1mH
- U2: footprint RTL2832U:QFN40P600X600X100-49N -> (none); Availability Not in stock -> (none); Check_prices https://www.snapeda.com/parts/RTL2832U/Realtek/view-part/?r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 -> (none); Description_1 DVB-T COFDM demodulator -> (none); MF Realtek Semiconductor Corp -> (none); Price None -> (none); SNAPEDA_PN RTL2832U -> (none); SnapEDA_Link https://www.snapeda.com/parts/RTL2832U/Realtek/view-part/?r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 -> (none)
Connections:
- net +3.3V: now also U2.14 (VDD3), U2.43 (VDDA33), U2.44 (VDDA), U2.47 (VDDA), U3.18 (VCC), C29.1, C30.1, C41.1, C50.1, C52.1, C53.1, C55.2, C56.2, R18.2, R20.1, U6.16 (GND), U6.3 (3.3V)
- net GND: now also U2.15 (AGC_RF), U2.8 (GNDPLL), C28.2, C29.2, C30.2, C41.2, C44.1, C46.2, C49.1, C50.2, C51.2, C52.2, C53.2, C55.1, C56.1, C57.1, U6.1 (GND), U6.2 (GND), U6.9 (GND)
- net GPIO10: now also U6.15 (CS-NSS)
- net GPIO11: now also U6.14 (MOSI)
- net GPIO12: now also U6.12 (SCK)
- net GPIO13: now also U6.13 (MISO)
- net GPIO14: now also U6.5 (DI00)
- net GPIO17: now also C57.2, R20.2, U6.4 (RESET)
- net USBD+: now also U2.40 (USB_D+_(HSDP))
- net USBD-: now also U2.41 (USB_D−_(HSDM))
- net at R16.2, R17.2, U2.17 (I2C_SDAT): now also C46.1
- net at R14.2, R15.2, U2.16 (I2C_SCLT): now also C44.2
- net +1V2: now reaches U2.12 (VDD1)
- net +1V2: now also U2.20 (VDD1), U2.28 (VDD1), U2.7 (VDDPLL), C49.2, C51.1
- net at U2.46 (VCMI): now also C28.1
- net at U2.48 (R12K): now also C54.1
- net at U2.9 (TP_CKO): now also J6.1 (Pin_1)
- net at U3.15 (CP): now also R19.2
- net at U3.17 (VDD_PLL): now also C47.2
- new net: C47.1, C48.2
- new net: C54.2, R18.1
- new net: C48.1, R19.1
- no-connect marks 14 -> 19
Other:
- note added: "GND guard with more via"
- note added: "Pin16 is PLL reference GND, please don't connect pin16 to E-PAD"
- note added: "mistake on diagram pin40 and 41 swapt"
- moved on the sheet: AE1, C10, C11, C12, C13, C14, C15, C16, C17, C18, C19, C20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

Commit message: Updating PCB to final design and updating partlist
Parts:
- removed C10, C13: 27pF, symbol Device:C_Small
- removed C17, C21: 100nF 16v Cer, symbol Device:C_Polarized_Small
- removed C18: 47pF, symbol Device:C_Small
- removed C54: 1uF, symbol Device:C_Small
- removed C55, C57: 100nF, symbol Device:C_Small
- removed D3, D4: Diod, symbol Device:D_Small
- removed J15: I/O Connector, Connector_PinHeader_2.54mm:PinHeader_2x08_P2.54mm_Vertical, symbol Connector_Generic:Conn_02x08_Odd_Even
- removed J16: Screw_Terminal_01x03, TerminalBlock:TerminalBlock_bornier-3_P5.08mm, symbol Connector:Screw_Terminal_01x03
- removed J17: Screw_Terminal_01x04, TerminalBlock:TerminalBlock_bornier-4_P5.08mm, symbol Connector:Screw_Terminal_01x04
- removed J5: Conn_Coaxial, symbol Connector:Conn_Coaxial
- removed L9: beet, symbol Device:L_Ferrite_Small
- removed R1, R6: 10k, symbol Device:R_Small
- removed R13: 101, symbol Device:R_Small
- removed R20: 220, Resistor_SMD:R_0805_2012Metric_Pad1.20x1.40mm_HandSolder, symbol Device:R_Small
- removed Y2: 16MHz, symbol Device:Crystal_Small
- removed Y3: 28.8Mhz, symbol Device:Crystal_Small
- added C14, C22: 132nF, Capacitor_SMD:C_0805_2012Metric, symbol Device:C_Small
- added C16: 47uF, Capacitor_SMD:C_1206_3216Metric, symbol Device:C_Small
- added C25, C26, C37, C39, C65, C69, C71, C72, C77: 100nF, Capacitor_SMD:C_0805_2012Metric, symbol Device:C_Small
- added C33: 2.2uF, Capacitor_SMD:C_0805_2012Metric, symbol Device:C_Small
- added C4: 330pF, Capacitor_SMD:C_0805_2012Metric, symbol Device:C_Small
- added C50: 10uF, Capacitor_SMD:C_0805_2012Metric, symbol Device:C_Polarized_Small
- added C51, C61: 100nF, Capacitor_SMD:C_0805_2012Metric, symbol Device:C_Polarized_Small
- added C52: 10nF, Capacitor_SMD:C_0805_2012Metric, symbol Device:C_Polarized_Small
- added C62: 2.2uF, Capacitor_SMD:C_0805_2012Metric, symbol Device:C_Polarized_Small
- added C63, C76: 22pF, Capacitor_SMD:C_0805_2012Metric, symbol Device:C_Small
- added C64, C67, C70, C74, C78: 1uF, Capacitor_SMD:C_0805_2012Metric, symbol Device:C_Small
- added C66, C73, C75: 10uF, Capacitor_SMD:C_0805_2012Metric, symbol Device:C_Small
- added D3, D6: VSSAF5M6HM3/H, Diode_SMD:D_SMA, symbol Device:D_Schottky_Small
- added D4, D5: 7012X5, LED_SMD:LED_0805_2012Metric, symbol Device:LED_Small
- added D7: 1N4007FL, Diode_SMD:D_SOD-123, symbol Diode:1N4148W
- added FB1, FB2: Bead, Capacitor_SMD:C_0805_2012Metric, symbol Device:FerriteBead_Small
- added IC2: BQ24650RVAR, BQ24650RVAR:QFN50P350X350X100-17N-D, symbol BQ24650RVAR:BQ24650RVAR
- added J1: CON-SMA-EDGE-S, CON_SMA_EDGE_S:RFSOLUTIONS_CON-SMA-EDGE-S, symbol CON_SMA_EDGE_S:CON-SMA-EDGE-S
- added J11: Solar connector, TB007_508_02BE:CUI_TB007-508-02BE, symbol Connector:Conn_01x02_Pin
- added J12: TS Conn, Connector_PinHeader_2.54mm:PinHeader_1x03_P2.54mm_Vertical, symbol Connector:Conn_01x03_Pin
- added J13: Conn_01x03_Pin, Jumper:SolderJumper-3_P1.3mm_Bridged12_RoundedPad1.0x1.5mm, symbol Connector:Conn_01x03_Pin
- added J14: BAT connector, TB007_508_02BE:CUI_TB007-508-02BE, symbol Connector:Conn_01x02_Pin
- added J8: Conn, Connector_PinHeader_2.54mm:PinHeader_1x04_P2.54mm_Vertical, symbol Connector:Conn_01x04_Pin
- added JP1, JP4, JP5: SolderJumper_2_Open, Jumper:SolderJumper-2_P1.3mm_Open_RoundedPad1.0x1.5mm, symbol Jumper:SolderJumper_2_Open
- added L1: 100nH, Inductor_SMD:L_0805_2012Metric, symbol Device:L
- added L15, L17: PIS150H-471M, PIS150H-471M:PIS150H471M, symbol PIS150H-471M:PIS150H-471M
- added L16: 10uH, IHLP2525CZER100M01:IND_IHLP_2525_CZ_VIS, symbol Device:L
- added L5, L9: 118.1nH, Inductor_SMD:L_0603_1608Metric, symbol Device:L_Small
- added L6, L8: 478nH, Inductor_SMD:L_0603_1608Metric, symbol Device:L_Small
- added L7: 470uH, SRR1260-471K:SRR12604R7Y, symbol Device:L
- added Q1, Q2: AO3407A, Package_TO_SOT_SMD:SOT-23, symbol Transistor_FET:AO3401A
- added Q3: SI7540DP-T1-GE3, SI7288DP-T1-GE3:TRANS_SI7540DP-T1-GE3, symbol SI7288DP-T1-GE3:SI7540DP-T1-GE3
- added R11: 1K, Resistor_SMD:R_0805_2012Metric, symbol Device:R_Small
- added R12, R38, R44: 100K, Resistor_SMD:R_0805_2012Metric, symbol Device:R_Small
- added R14, R39: 220, Resistor_SMD:R_0805_2012Metric, symbol Device:R_Small
- added R18, R37: 100, Resistor_SMD:R_0805_2012Metric, symbol Device:R_Small
- added R24: 0 Ohm, Resistor_SMD:R_0805_2012Metric, symbol Device:R_Small
- added R30, R35, R40: 10K, Resistor_SMD:R_0805_2012Metric, symbol Device:R_Small
- added R31, R43: 499K, Resistor_SMD:R_0805_2012Metric, symbol Device:R_Small
- added R32: 36K, Resistor_SMD:R_0805_2012Metric, symbol Device:R_Small
- added R33: 5K23, Resistor_SMD:R_0805_2012Metric, symbol Device:R_Small
- added R34: 30K1, Resistor_SMD:R_0805_2012Metric, symbol Device:R_Small
- added R36: 10, Resistor_SMD:R_0805_2012Metric, symbol Device:R_Small
- added R41: 2.2, Resistor_SMD:R_0805_2012Metric, symbol Device:R_Small
- added R42: 0.033, Resistor_SMD:R_1206_3216Metric, symbol Device:R_Small
- added T1: TCM1-382WX+, TCM1-382WX+:TCM1382WX, symbol TCM1-382WX+:TCM1-382WX+
- added U1: BAV99-7-F, BAV99-7-F:SOT-23_DIO, symbol BAV99-7-F:BAV99-7-F
- added Y1: 28.8MHz, ATX11F32000MHZF05T, symbol ATX-11-F-32.000MHZ-F05-T:ATX-11-F-32.000MHZ-F05-T
- C1: renamed from C3; footprint (none) -> Capacitor_SMD:C_0805_2012Metric
- C10: renamed from C26; footprint (none) -> Capacitor_SMD:C_0805_2012Metric
- C11: renamed from C5; footprint Capacitor_SMD:C_0805_2012Metric_Pad1.18x1.45mm_HandSolder -> Capacitor_SMD:C_0805_2012Metric
- C12: renamed from C30; value 105 -> 100nF; footprint (none) -> Capacitor_SMD:C_0805_2012Metric
- C13: renamed from C4; footprint Capacitor_SMD:C_0805_2012Metric_Pad1.18x1.45mm_HandSolder -> Capacitor_SMD:C_0805_2012Metric
- C15: renamed from C6; footprint Capacitor_SMD:C_0805_2012Metric_Pad1.18x1.45mm_HandSolder -> Capacitor_SMD:C_0805_2012Metric
- C17: renamed from C7; footprint Capacitor_SMD:C_0805_2012Metric_Pad1.18x1.45mm_HandSolder -> Capacitor_SMD:C_0805_2012Metric
- C18: renamed from C8; value 105 -> 1uF; footprint (none) -> Capacitor_SMD:C_0805_2012Metric
- C19: value 47pF -> 212nF; footprint (none) -> Capacitor_SMD:C_0805_2012Metric
- C2: renamed from C29; value 105 -> 100nF; footprint (none) -> Capacitor_SMD:C_0805_2012Metric
- C20: renamed from C9; value 104 -> 100nF; footprint (none) -> Capacitor_SMD:C_0805_2012Metric
- C21: renamed from C27; footprint (none) -> Capacitor_SMD:C_0805_2012Metric
- C23: renamed from C11; footprint Capacitor_SMD:C_0805_2012Metric_Pad1.18x1.45mm_HandSolder -> Capacitor_SMD:C_0805_2012Metric
- C24: renamed from C12; footprint Capacitor_SMD:C_0805_2012Metric_Pad1.18x1.45mm_HandSolder -> Capacitor_SMD:C_0805_2012Metric
- C27: renamed from C23; footprint Capacitor_SMD:C_0805_2012Metric_Pad1.18x1.45mm_HandSolder -> Capacitor_SMD:C_0805_2012Metric
- C28: renamed from C24; footprint Capacitor_SMD:C_0805_2012Metric_Pad1.18x1.45mm_HandSolder -> Capacitor_SMD:C_0805_2012Metric
- C29: renamed from C44; value 27pF -> 39pF; footprint (none) -> Capacitor_SMD:C_0805_2012Metric
- C3: renamed from C41; value 105 -> 10nF; footprint (none) -> Capacitor_SMD:C_0805_2012Metric
- C30: renamed from C46; value 27pF -> 39pF; footprint (none) -> Capacitor_SMD:C_0805_2012Metric
- C31: renamed from C51; footprint (none) -> Capacitor_SMD:C_0805_2012Metric
- C32: renamed from C25; value 27pF -> 100nF; footprint (none) -> Capacitor_SMD:C_0805_2012Metric
- C34: renamed from C15; value 22uF 16v Cer -> 10uF; footprint (none) -> Capacitor_SMD:C_0805_2012Metric
- C35: renamed from C22; value 27pF -> 100nF; footprint (none) -> Capacitor_SMD:C_0805_2012Metric
- C36: renamed from C50; footprint (none) -> Capacitor_SMD:C_0805_2012Metric
- C38: renamed from C49; footprint (none) -> Capacitor_SMD:C_0805_2012Metric
- C5: renamed from C47; value 1Uf -> 100nF; footprint (none) -> Capacitor_SMD:C_0805_2012Metric
- C53: renamed from C42; value C_Small -> 1.5pF
- C54: renamed from C43; value C_Small -> 1.5pF
- C55: renamed from C28; footprint (none) -> Capacitor_SMD:C_0805_2012Metric
- C56: renamed from C20; value 100nF 16v Cer -> 100nF; footprint (none) -> Capacitor_SMD:C_0805_2012Metric
- C57: renamed from C53; footprint (none) -> Capacitor_SMD:C_0805_2012Metric
- C58: renamed from C45; value C_Small -> 1.5pF
- C59: renamed from C16; value 10uF 16v Cer -> 10uF; footprint (none) -> Capacitor_SMD:C_0805_2012Metric
- C6: renamed from C48; value 1Uf -> 6n8F; footprint (none) -> Capacitor_SMD:C_0805_2012Metric
- C60: renamed from C52; footprint (none) -> Capacitor_SMD:C_0805_2012Metric
- C68: renamed from C56; footprint (none) -> Capacitor_SMD:C_0805_2012Metric
- C7: renamed from C1; footprint Capacitor_SMD:C_0805_2012Metric_Pad1.18x1.45mm_HandSolder -> Capacitor_SMD:C_0805_2012Metric
- C8: renamed from C2; footprint Capacitor_SMD:C_0805_2012Metric_Pad1.18x1.45mm_HandSolder -> Capacitor_SMD:C_0805_2012Metric
- C9: renamed from C14; value 104 -> 100nF; footprint (none) -> Capacitor_SMD:C_0805_2012Metric
- D1, D2: value 1N4148W -> 1N4007FL
- J2: renamed from J1; footprint TerminalBlock:TerminalBlock_bornier-2_P5.08mm -> TB007_508_02BE:CUI_TB007-508-02BE
- J7: renamed from J6; footprint (none) -> Connector_PinHeader_2.54mm:PinHeader_1x01_P2.54mm_Vertical
- L10: renamed from L1; footprint Inductor_SMD:L_0805_2012Metric_Pad1.15x1.40mm_HandSolder -> Inductor_SMD:L_0805_2012Metric
- L11: renamed from L8; value 4.7uH -> 10uH; footprint (none) -> Inductor_SMD:L_0805_2012Metric
- L13: renamed from L3; value L_Small -> 2.7nH
- L14: renamed from L4; value L_Small -> 2.7nH
- L2: renamed from L5; value 1mH -> 8n2H; footprint (none) -> Inductor_SMD:L_0805_2012Metric
- L3: renamed from L6; footprint (none) -> Inductor_SMD:L_0805_2012Metric
- L4: renamed from L7; footprint (none) -> Inductor_SMD:L_0805_2012Metric
- R1: renamed from R19; value 1K -> 1K8; footprint (none) -> Resistor_SMD:R_0805_2012Metric
- R10: renamed from R14; value 220 -> 22; footprint (none) -> Resistor_SMD:R_0805_2012Metric
- R13: renamed from R7; footprint Resistor_SMD:R_0805_2012Metric_Pad1.20x1.40mm_HandSolder -> Resistor_SMD:R_0805_2012Metric
- R15: renamed from R11; footprint Resistor_SMD:R_0805_2012Metric_Pad1.20x1.40mm_HandSolder -> Resistor_SMD:R_0805_2012Metric
- R16: renamed from R12; footprint Resistor_SMD:R_0805_2012Metric_Pad1.20x1.40mm_HandSolder -> Resistor_SMD:R_0805_2012Metric
- R17: renamed from R15; value 472 -> 4K7; footprint (none) -> Resistor_SMD:R_0805_2012Metric
- R19: renamed from R22; footprint Resistor_SMD:R_0805_2012Metric_Pad1.20x1.40mm_HandSolder -> Resistor_SMD:R_0805_2012Metric
- R2: renamed from R10; value 103 -> 10K; footprint (none) -> Resistor_SMD:R_0805_2012Metric
- R20: renamed from R17; value 472 -> 4K7; footprint (none) -> Resistor_SMD:R_0805_2012Metric
- R21: renamed from R23; footprint Resistor_SMD:R_0805_2012Metric_Pad1.20x1.40mm_HandSolder -> Resistor_SMD:R_0805_2012Metric
- R22: renamed from R26; footprint Resistor_SMD:R_0805_2012Metric_Pad1.20x1.40mm_HandSolder -> Resistor_SMD:R_0805_2012Metric
- R23: renamed from R27; footprint Resistor_SMD:R_0805_2012Metric_Pad1.20x1.40mm_HandSolder -> Resistor_SMD:R_0805_2012Metric
- R25: renamed from R33; footprint Resistor_SMD:R_0805_2012Metric_Pad1.20x1.40mm_HandSolder -> Resistor_SMD:R_0805_2012Metric
- R26: renamed from R34; footprint Resistor_SMD:R_0805_2012Metric_Pad1.20x1.40mm_HandSolder -> Resistor_SMD:R_0805_2012Metric
- R27: renamed from R36; footprint Resistor_SMD:R_0805_2012Metric_Pad1.20x1.40mm_HandSolder -> Resistor_SMD:R_0805_2012Metric
- R28: renamed from R18; value 10k -> 10K; footprint (none) -> Resistor_SMD:R_0805_2012Metric
- R29: renamed from R37; footprint Resistor_SMD:R_0805_2012Metric_Pad1.20x1.40mm_HandSolder -> Resistor_SMD:R_0805_2012Metric
- R3: renamed from R2; footprint Resistor_SMD:R_0805_2012Metric_Pad1.20x1.40mm_HandSolder -> Resistor_SMD:R_0805_2012Metric
- R4: renamed from R3; value 0 -> 0 Ohm; footprint Resistor_SMD:R_0805_2012Metric_Pad1.20x1.40mm_HandSolder -> Resistor_SMD:R_0805_2012Metric
- R5: renamed from R4; value 0 -> 0 Ohm; footprint Resistor_SMD:R_0805_2012Metric_Pad1.20x1.40mm_HandSolder -> Resistor_SMD:R_0805_2012Metric
- R6: renamed from R5; footprint Resistor_SMD:R_0805_2012Metric_Pad1.20x1.40mm_HandSolder -> Resistor_SMD:R_0805_2012Metric
- R7: renamed from R16; value 220 -> 22; footprint (none) -> Resistor_SMD:R_0805_2012Metric
- R8, R9: value 220 -> 22; footprint (none) -> Resistor_SMD:R_0805_2012Metric
- U5: renamed from U2; footprint (none) -> RTL2832U:QFN40P600X600X100-49N
- renumbered C31 to C40, C32 to C41, C33 to C42, C34 to C43, C35 to C44, C36 to C45, C37 to C46, C38 to C47, C39 to C48, C40 to C49, J12 to J10, J13 to J3, J2 to J4, J3 to J5, J4 to J6, J10 to J9, JP6 to JP2, JP8 to JP3, L2 to L12, U1 to U2, U5 to U6, U6 to U7, Y1 to Y2
Connections:
- net +15V: now also D7.1 (K)
- net +1V2: now also C34.1, C57.1, L11.1, U5.34 (VDD1), U5.42 (UVDDA), U5.44 (VDDA), U5.47 (VDDA), C61.1, C62.1, FB1.1, R24.1; no longer C38.2, U5.7 (VDDPLL)
- net +3.3V: now also C26.2, C65.2, L7.2, Q1.2 (S), Q2.2 (S), R12.2, R38.2; no longer C10.1, C11.2, C12.1, C2.1, C3.1, C36.1, C57.1, C60.1, C68.2, IC1.2 (OUTPUT), IC1.4 (VOUT), R17.1, R20.1, R28.2, U3.11 (VCC), U3.18 (VCC), U3.2 (VCC), U3.23 (VCC), U5.14 (VDD3), U5.43 (VDDA33), U5.44 (VDDA), U5.47 (VDDA), U6.8 (VCC), U7.16 (GND), U7.3 (3.3V)
- net +5V: now also L1.2; no longer J3.4 (Pin_4)
- net GND: now also C19.2, C5.1, C6.1, R28.2, U5.3 (GNDA), U5.39 (SEGND), U5.45 (GNDA), U6.7 (~{WC}), U7.16 (GND), C14.2, C16.1, C22.2, C25.1, C33.1, C4.1, C50.2, C51.2, C52.2, C61.2, C62.2, C66.1, C70.1, C73.1, C74.2, C75.1, C78.1, IC2.11 (GND), IC2.17 (EP), IC2.19 (VIA_B), J1.G1, J1.G2, J1.G3, J1.G4, J11.2 (Pin_2), J14.2 (Pin_2), J8.4 (Pin_4), Q3.3, T1.1 (GND_1), T1.2 (GND_2), U1.1 (EPAD), U1.2 (EPAD), Y1.2 (GND); no longer C19.1, U5.15 (AGC_RF), U7.1 (GND)
- net GNDA: now also C64.1, C67.1, C72.2, C77.1, IC2.18 (VIA_A), J12.1 (Pin_1), J13.3 (Pin_3), R30.2, R32.1, R34.1, R44.1; no longer U5.3 (GNDA), U5.45 (GNDA)
- net GPIO1: now also R12.1, R14.1
- net GPIO10: now also U7.4 (RESET); no longer U7.15 (CS-NSS)
- net GPIO11: now also U7.5 (DI00); no longer U7.14 (MOSI)
- net GPIO12: now also U7.6 (DI01); no longer U7.12 (SCK)
- net GPIO13: now also U7.7 (DI02); no longer U7.13 (MISO)
- net GPIO14: now also U7.8 (DI03); no longer U7.5 (DI00)
- net GPIO15: now also R38.1, R39.1
- net GPIO17: no longer U7.4 (RESET)
- net GPIO2/PTT ESP: no longer U4.7 (GPIO2)
- net GPIO3: now also U7.14 (MOSI)
- net GPIO4/BCLK: now also U7.13 (MISO)
- net GPIO5/FSYNC: now also U7.12 (SCK)
- net GPIO6/DOUT: now also U7.11 (DI05)
- net GPIO7/DIN: now also U7.10 (DI04)
- net at C56.1, C59.1, U5.25 (SW_VDD3)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: now also FB2.1
- net at C6.2: now also R1.1; no longer C5.1
- net at C1.2, L2.1: now also U1.3 (EPAD)
- net at U5.48 (R12K): now also R28.1
- net at R2.2, U5.13 (AGC_IF): now also R11.1
- net at R1.2, U3.15 (CP): now also C4.2
- net at U5.11 (XI): now also R18.2; no longer C21.2
- net 3.3V: now reaches U5.33 (VDD3)
- net 3.3V: now also C10.1, C12.1, C2.1, C3.1, C36.1, C60.1, R17.1, R20.1, U3.11 (VCC), U3.18 (VCC), U3.2 (VCC), U3.23 (VCC), U5.14 (VDD3), U5.43 (VDDA33), U6.8 (VCC), C25.2, C50.1, C51.1, C52.1, FB2.2, J8.1 (Pin_1), Q1.3 (D), R11.2, Y1.1 (OE), Y1.4 (VDD)
- net at U5.4 (VQP): now also C39.2
- net at U5.5 (VQN): now also C37.2
- net at U3.8 (XTAL_I): now also Y1.3 (OUT)
- net at C1.1: now also J1.1, JP1.1 (A)
- net at U3.3 (LT): now also L5.1
- new net: D3.2 (A), JP4.1 (A), L15.3, L15.4
- new net: C76.2, C77.2, C78.2, D7.2 (A), J14.1 (Pin_1), JP5.1 (A), L17.3, L17.4, R43.2
- new net: R24.2, U5.23 (FB)
- new net: C11.2, C16.2, IC1.2 (OUTPUT), IC1.4 (VOUT), L7.1
- new net: C14.1, L5.2, L6.1
- new net: C63.1, IC2.2 (MPPSET), R31.1, R32.2
- new net: C26.1, Q1.1 (G), R14.2
- new net: C64.2, IC2.1 (VCC), R36.2
- new net: C70.2, D6.2 (A), IC2.12 (REGN)
- new net: C69.2, IC2.14 (PH), L16.1, Q3.1, Q3.10, Q3.5, Q3.6
- new net: IC2.15 (HIDRV), Q3.2
- new net: IC2.13 (LODRV), Q3.4
- new net: C73.2, C74.1, D3.1 (K), Q3.7, Q3.8, Q3.9, R36.1
- new net: C33.2, C38.2, FB1.2, U5.7 (VDDPLL)
- new net: C22.1, L8.2, L9.1
- new net: C71.2, C75.2, IC2.9 (SRN), JP5.2 (B), L17.1, L17.2, R42.1
- new net: D4.2 (A), R35.1
- new net: C71.1, C72.1, IC2.10 (SRP), L16.2, R42.2
- new net: JP1.2 (B), L1.1
- new net: C37.1, J8.2 (Pin_2), T1.5 (SECONDARY_DOT)
- new net: D5.1 (K), IC2.5 (STAT2)
- new net: D5.2 (A), R40.1
- new net: L9.2, T1.3 (PRIMARY_DOT)
- new net: C39.1, J8.3 (Pin_3), T1.4 (SECONDARY)
- new net: C69.1, D6.1 (K), R41.2
- new net: IC2.16 (BTST), R41.1
- new net: D4.1 (K), IC2.3 (STAT1)
- new net: IC2.4 (TS), R37.2
- new net: IC2.7 (TERM_EN), J13.2 (Pin_2)
- new net: C76.1, IC2.8 (VFB), R43.1, R44.2
- new net: C19.1, L6.2, L8.1
- new net: C21.2, R18.1
- new net: J12.2 (Pin_2), R33.1, R34.2, R37.1
- new net: J12.3 (Pin_3), R30.1
- new net: C66.2, C68.2, Q2.3 (D), U7.3 (3.3V)
- new net: C65.1, Q2.1 (G), R39.2
- new net +16V: C63.2, J11.1 (Pin_1), JP4.2 (B), L15.1, L15.2, R31.2
- new net GPIO2: U4.7 (GPIO2), U7.15 (CS-NSS)
- new net VREF: C67.2, IC2.6 (VREF), J13.1 (Pin_1), R33.2, R35.2, R40.2
- no-connect marks 19 -> 31
Other:
- note added: "3.3V ref voltage output"
- note added: "Bring out Q+ Q- to connector"
- note added: "Confirm ESP32-S3 OTG Mode Selection"
- note added: "LoRa Device"
- note added: "VOUT"
- note removed: "Check connections"
- note removed: "EXP GND"
- note removed: "Mic GND"
- note removed: "PTT"
- note removed: "PTT Power"
- note removed: "PTTGND"
- note removed: "Radio EXP"
- note removed: "Radio Mic"
- moved on the sheet: C1, C11, C2, C21, C3, C32, C34, C35, C36, C38, C5, C56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
